File: PCB/arnaansRealMacropad.kicad_pcb (KiCad board)
At the start: 2 copper layers, 94.8 x 79 mm, 22 parts, among them J1 Conn_01x04_Pin, SW1 SW_Push_45deg, SW2 SW_Push_45deg, SW3 SW_Push_45deg, SW4 SW_Push_45deg, SW5 SW_Push_45deg, SW6 SW_Push_45deg, SW7 RotaryEncoder_Switch, U1 MOUDLE-SEEEDUINO-XIAO

Commit message: Fixed LED footprint
Parts:
- D10, D8, D9: footprint LED_SMD:LED_SK6812MINI_PLCC4_3.5x3.5mm_P1.75mm -> footprints:SK6812MINI-E_fixed; moved to B.Cu
- turned D10 to 180 degrees
- turned D8 to 180 degrees
- turned D9 to 180 degrees
Routing:
- net Net-(D8-DOUT): track 26.8 -> 8.47 mm, vias 2 -> 0
- net GND: track 194.7 -> 184.3 mm
- net Net-(D10-DIN): track 14.6 -> 5.83 mm
- net WS2812B: track 87.7 -> 92.6 mm
- net VCC: track 159.1 -> 161.8 mm
