File: PCB/arnaansRealMacropad.kicad_sch (KiCad schematic)
At the start: 19 parts, among them J1 Conn_01x04_Pin, SW1 SW_Push_45deg, SW2 SW_Push_45deg, SW3 SW_Push_45deg, SW4 SW_Push_45deg, SW5 SW_Push_45deg, SW6 SW_Push_45deg, SW7 RotaryEncoder_Switch, U1 MOUDLE-SEEEDUINO-XIAO

Commit message: Fixed LED footprint
Parts:
- D10, D8, D9: footprint LED_SMD:LED_SK6812MINI_PLCC4_3.5x3.5mm_P1.75mm -> footprints:SK6812MINI-E_fixed
Changed lines of the file:
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@@
 			)
 		)
-		(property "Footprint" "LED_SMD:LED_SK6812MINI_PLCC4_3.5x3.5mm_P1.75mm"
+		(property "Footprint" "footprints:SK6812MINI-E_fixed"
 			(at 124.46 130.81 0)
 			(effects
@@
 			)
 		)
-		(property "Footprint" "LED_SMD:LED_SK6812MINI_PLCC4_3.5x3.5mm_P1.75mm"
+		(property "Footprint" "footprints:SK6812MINI-E_fixed"
 			(at 48.26 130.81 0)
 			(effects
@@
 			)
 		)
-		(property "Footprint" "LED_SMD:LED_SK6812MINI_PLCC4_3.5x3.5mm_P1.75mm"
+		(property "Footprint" "footprints:SK6812MINI-E_fixed"
 			(at 86.36 130.81 0)
 			(effects
